File: FG-VCO-(core1)/FG-VCO-(core1).kicad_pcb (KiCad board)
At the start: 2 copper layers, 53.3 x 106.7 mm, 72 parts, among them J1 conn_signals_out, J10 conn_signals_in_3, J2 conn_power_out, J3 conn_modulation, J4 conn_power_in, J5 conn_signals_in_1, J6 Exponential Test, J7 Test CLK, J8 conn_mode, J9 conn_signals_in_2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

Commit message: same as previous, for the whole folder
Parts:
- removed C8: 10n, Custom Footprints:C_Disc_P2.54mm
- added J15: VFC out, Connector_PinHeader_2.54mm:PinHeader_1x01_P2.54mm_Vertical, F.Cu at (26.7, 40.0)
- RV1: footprint Potentiometer_THT:Potentiometer_Bourns_3339P_Vertical_HandSoldering -> Potentiometer_THT:Potentiometer_Vishay_T73YP_Vertical
- moved R12 7.62 mm to (5.71, 14.6), turned to -90 degrees
- moved J9 6.35 mm to (10.2, 98.4)
- moved RV1 5.08 mm to (43.2, 33.7), turned to 90 degrees
- moved J4 0.64 mm to (22.9, 3.81)
- moved J2 0.64 mm to (22.9, 1.27)
Connections:
- RV1 pad 1: +12V -> GNDD
- RV1 pad 3: GNDD -> +12V
Routing:
- net Sine_in: track 25.0 -> 31.5 mm
- net Triangle_in: track 12.8 -> 19.1 mm
- net Square_in: track 8.19 -> 14.5 mm
- net +5V: track 208.6 -> 207.3 mm
- net -12V: track 187.8 -> 188.7 mm
Other:
- outline, holes or cut-outs redrawn
