File: FG-VCO-(core1)/monostable_circuit.kicad_sch (KiCad schematic)
At the start: 4 parts, among them U6 NE555D

Commit message: same as previous, for the whole folder
Changed lines of the file:
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@@
+    (stroke (width 0) (type default) (color 0 0 0 0))
+  )
+  (wire (pts (xy 88.9 82.55) (xy 114.3 82.55))
     (stroke (width 0) (type default) (color 0 0 0 0))
   )
@@
     (stroke (width 0) (type default) (color 0 0 0 0))
   )
-  (wire (pts (xy 88.9 82.55) (xy 114.3 82.55))
-    (stroke (width 0) (type default) (color 0 0 0 0))
-  )
-  (wire (pts (xy 139.7 82.55) (xy 165.1 82.55))
+  (wire (pts (xy 139.7 82.55) (xy 177.8 82.55))
     (stroke (width 0) (type default) (color 0 0 0 0))
   )
@@
     (stroke (width 0) (type default) (color 0 0 0 0))
   )
-  (hierarchical_label "pulse_out" (shape output) (at 165.1 82.55 0)
+  (hierarchical_label "pulse_out" (shape output) (at 177.8 82.55 0)
     (effects (font (size 1.27 1.27)) (justify left))
   )
