File: FG-VCO-(core1)/v_f_conv.kicad_sch (KiCad schematic)
At the start: 5 parts, among them U5 VFC110

Commit message: same as previous, for the whole folder
Parts:
- removed C8: 10n, Custom Footprints:C_Disc_P2.54mm, symbol Device:C
- added J15: VFC out, Connector_PinHeader_2.54mm:PinHeader_1x01_P2.54mm_Vertical, symbol Connector:Conn_01x01_Male
Connections:
- net f_out: now also J15.1 (Pin_1)
Changed lines of the file:
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@@
   (junction (at 99.06 81.28) (diameter 0) (color 0 0 0 0)
   )
-  (junction (at 152.4 68.58) (diameter 0) (color 0 0 0 0)
+  (junction (at 165.1 81.28) (diameter 0) (color 0 0 0 0)
   )
   (junction (at 152.4 81.28) (diameter 0) (color 0 0 0 0)
@@
   (no_connect (at 144.78 93.98))
   (no_connect (at 144.78 86.36))
+  (wire (pts (xy 165.1 81.28) (xy 177.8 81.28))
+    (stroke (width 0) (type default) (color 0 0 0 0))
+  )
   (wire (pts (xy 116.84 73.66) (xy 121.92 73.66))
     (stroke (width 0) (type default) (color 0 0 0 0))
@@
     (stroke (width 0) (type default) (color 0 0 0 0))
   )
-  (wire (pts (xy 152.4 81.28) (xy 184.15 81.28))
-    (stroke (width 0) (type default) (color 0 0 0 0))
-  )
-  (wire (pts (xy 165.1 68.58) (xy 165.1 71.12))
-    (stroke (width 0) (type default) (color 0 0 0 0))
-  )
-  (wire (pts (xy 152.4 68.58) (xy 152.4 71.12))
-    (stroke (width 0) (type default) (color 0 0 0 0))
-  )
-  (wire (pts (xy 152.4 68.58) (xy 154.94 68.58))
+  (wire (pts (xy 152.4 81.28) (xy 165.1 81.28))
     (stroke (width 0) (type default) (color 0 0 0 0))
   )
@@
     (stroke (width 0) (type default) (color 0 0 0 0))
   )
-  (wire (pts (xy 152.4 66.04) (xy 152.4 68.58))
+  (wire (pts (xy 152.4 66.04) (xy 152.4 71.12))
     (stroke (width 0) (type default) (color 0 0 0 0))
   )
@@
     (stroke (width 0) (type default) (color 0 0 0 0))
   )
+  (wire (pts (xy 76.2 63.5) (xy 116.84 63.5))
+    (stroke (width 0) (type default) (color 0 0 0 0))
+  )
   (wire (pts (xy 109.22 86.36) (xy 109.22 88.9))
     (stroke (width 0) (type default) (color 0 0 0 0))
@@
     (stroke (width 0) (type default) (color 0 0 0 0))
   )
-  (wire (pts (xy 82.55 63.5) (xy 116.84 63.5))
-    (stroke (width 0) (type default) (color 0 0 0 0))
-  )
-  (wire (pts (xy 162.56 68.58) (xy 165.1 68.58))
-    (stroke (width 0) (type default) (color 0 0 0 0))
-  )
   (wire (pts (xy 144.78 81.28) (xy 152.4 81.28))
     (stroke (width 0) (type default) (color 0 0 0 0))
@@
     (stroke (width 0) (type default) (color 0 0 0 0))
   )
+  (wire (pts (xy 165.1 81.28) (xy 165.1 119.38))
+    (stroke (width 0) (type default) (color 0 0 0 0))
+  )
   (wire (pts (xy 119.38 91.44) (xy 119.38 93.98))
     (stroke (width 0) (type default) (color 0 0 0 0))
@@
     (stroke (width 0) (type default) (color 0 0 0 0))
   )
-  (hierarchical_label "f_out" (shape output) (at 184.15 81.28 0)
+  (hierarchical_label "f_out" (shape output) (at 177.8 81.28 0)
     (effects (font (size 1.27 1.27)) (justify left))
   )
-  (hierarchical_label "V_in" (shape input) (at 82.55 63.5 180)
+  (hierarchical_label "V_in" (shape input) (at 76.2 63.5 180)
     (effects (font (size 1.27 1.27)) (justify right))
   )
@@
     (pin "2")
   )
+  (symbol (lib_id "Connector:Conn_01x01_Male") (at 165.1 124.46 90) (unit 1)
+    (in_bom yes) (on_board yes) (fields_autoplaced)
+    (property "Reference" "J15" (id 0) (at 165.9382 122.9165 90)
+      (effects (font (size 1.27 1.27)) (justify right))
+    )
+    (property "Value" "VFC out" (id 1) (at 165.9382 125.6916 90)
+      (effects (font (size 1.27 1.27)) (justify right))
+    )
+    (property "Footprint" "Connector_PinHeader_2.54mm:PinHeader_1x01_P2.54mm_Vertical" (id 2) (at 165.1 124.46 0)
+      (effects (font (size 1.27 1.27)) hide)
+    )
+    (property "Datasheet" "~" (id 3) (at 165.1 124.46 0)
+      (effects (font (size 1.27 1.27)) hide)
+    )
+    (pin "1")
+  )
   (symbol (lib_id "Device:C") (at 109.22 92.71 180) (unit 1)
     (in_bom yes) (on_board yes) (fields_autoplaced)
@@
     (pin "1")
   )
-  (symbol (lib_id "power:GNDD") (at 165.1 71.12 0) (unit 1)
-    (in_bom yes) (on_board yes) (fields_autoplaced)
-    (property "Reference" "#PWR0135" (id 0) (at 165.1 77.47 0)
-      (effects (font (size 1.27 1.27)) hide)
-    )
-    (property "Value" "GNDD" (id 1) (at 165.1 75.3015 0))
-    (property "Footprint" "" (id 2) (at 165.1 71.12 0)
-      (effects (font (size 1.27 1.27)) hide)
-    )
-    (property "Datasheet" "" (id 3) (at 165.1 71.12 0)
-      (effects (font (size 1.27 1.27)) hide)
-    )
-    (pin "1")
-  )
-  (symbol (lib_id "Device:C") (at 158.75 68.58 90) (unit 1)
-    (in_bom yes) (on_board yes) (fields_autoplaced)
-    (property "Reference" "C8" (id 0) (at 158.75 62.4545 90))
-    (property "Value" "10n" (id 1) (at 158.75 65.2296 90))
-    (property "Footprint" "Custom Footprints:C_Disc_P2.54mm" (id 2) (at 162.56 67.6148 0)
-      (effects (font (size 1.27 1.27)) hide)
-    )
-    (property "Datasheet" "~" (id 3) (at 158.75 68.58 0)
-      (effects (font (size 1.27 1.27)) hide)
-    )
-    (pin "1")
-    (pin "2")
-  )
   (symbol (lib_id "power:+5V") (at 152.4 66.04 0) (unit 1)
