File: FG-VCO-(core1)/out_stage.kicad_sch (KiCad schematic)
At the start: 25 parts, among them U7 TL074, U8 TL074

Commit message: finished ch06 and added appendix
Parts:
- C11, C12, C13, C14, C15: value 47p -> 30p
Changed lines of the file:
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@@
     (in_bom yes) (on_board yes) (fields_autoplaced)
     (property "Reference" "C12" (id 0) (at 63.5 63.7245 90))
-    (property "Value" "47p" (id 1) (at 63.5 66.4996 90))
+    (property "Value" "30p" (id 1) (at 63.5 66.4996 90))
     (property "Footprint" "Custom Footprints:C_Disc_P2.54mm" (id 2) (at 67.31 68.8848 0)
       (effects (font (size 1.27 1.27)) hide)
@@
     (in_bom yes) (on_board yes) (fields_autoplaced)
     (property "Reference" "C14" (id 0) (at 165.1 21.8145 90))
-    (property "Value" "47p" (id 1) (at 165.1 24.5896 90))
+    (property "Value" "30p" (id 1) (at 165.1 24.5896 90))
     (property "Footprint" "Custom Footprints:C_Disc_P2.54mm" (id 2) (at 168.91 26.9748 0)
       (effects (font (size 1.27 1.27)) hide)
@@
     (in_bom yes) (on_board yes) (fields_autoplaced)
     (property "Reference" "C15" (id 0) (at 165.1 66.2645 90))
-    (property "Value" "47p" (id 1) (at 165.1 69.0396 90))
+    (property "Value" "30p" (id 1) (at 165.1 69.0396 90))
     (property "Footprint" "Custom Footprints:C_Disc_P2.54mm" (id 2) (at 168.91 71.4248 0)
       (effects (font (size 1.27 1.27)) hide)
@@
     (in_bom yes) (on_board yes) (fields_autoplaced)
     (property "Reference" "C13" (id 0) (at 63.5 114.5245 90))
-    (property "Value" "47p" (id 1) (at 63.5 117.2996 90))
+    (property "Value" "30p" (id 1) (at 63.5 117.2996 90))
     (property "Footprint" "Custom Footprints:C_Disc_P2.54mm" (id 2) (at 67.31 119.6848 0)
       (effects (font (size 1.27 1.27)) hide)
@@
     (in_bom yes) (on_board yes) (fields_autoplaced)
     (property "Reference" "C11" (id 0) (at 63.5 19.2745 90))
-    (property "Value" "47p" (id 1) (at 63.5 22.0496 90))
+    (property "Value" "30p" (id 1) (at 63.5 22.0496 90))
     (property "Footprint" "Custom Footprints:C_Disc_P2.54mm" (id 2) (at 67.31 24.4348 0)
       (effects (font (size 1.27 1.27)) hide)
