File: FG-VCO-(core1)/sum_clip.kicad_sch (KiCad schematic)
At the start: 9 parts, among them U1 TL074

Commit message: same as previous, for the whole folder
Parts:
- RV1: footprint Potentiometer_THT:Potentiometer_Bourns_3339P_Vertical_HandSoldering -> Potentiometer_THT:Potentiometer_Vishay_T73YP_Vertical
Connections:
- net +12V: now also RV1.3; no longer RV1.1
- net GNDD: now also RV1.1; no longer RV1.3
Other:
- moved on the sheet: RV1
Changed lines of the file:
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@@
   (junction (at 102.87 73.66) (diameter 0) (color 0 0 0 0)
   )
+  (wire (pts (xy 127 76.2) (xy 121.92 76.2))
+    (stroke (width 0) (type default) (color 0 0 0 0))
+  )
+  (wire (pts (xy 127 76.2) (xy 127 85.09))
+    (stroke (width 0) (type default) (color 0 0 0 0))
+  )
+  (wire (pts (xy 102.87 73.66) (xy 106.68 73.66))
+    (stroke (width 0) (type default) (color 0 0 0 0))
+  )
+  (wire (pts (xy 177.8 86.36) (xy 173.99 86.36))
+    (stroke (width 0) (type default) (color 0 0 0 0))
+  )
+  (wire (pts (xy 177.8 86.36) (xy 177.8 90.17))
+    (stroke (width 0) (type default) (color 0 0 0 0))
+  )
+  (wire (pts (xy 83.82 81.28) (xy 87.63 81.28))
+    (stroke (width 0) (type default) (color 0 0 0 0))
+  )
+  (wire (pts (xy 177.8 74.93) (xy 177.8 86.36))
+    (stroke (width 0) (type default) (color 0 0 0 0))
+  )
+  (wire (pts (xy 162.56 86.36) (xy 166.37 86.36))
+    (stroke (width 0) (type default) (color 0 0 0 0))
+  )
+  (wire (pts (xy 76.2 81.28) (xy 72.39 81.28))
+    (stroke (width 0) (type default) (color 0 0 0 0))
+  )
+  (wire (pts (xy 72.39 77.47) (xy 72.39 81.28))
+    (stroke (width 0) (type default) (color 0 0 0 0))
+  )
+  (wire (pts (xy 110.49 63.5) (xy 102.87 63.5))
+    (stroke (width 0) (type default) (color 0 0 0 0))
+  )
+  (wire (pts (xy 99.06 63.5) (xy 102.87 63.5))
+    (stroke (width 0) (type default) (color 0 0 0 0))
+  )
+  (wire (pts (xy 102.87 53.34) (xy 102.87 63.5))
+    (stroke (width 0) (type default) (color 0 0 0 0))
+  )
+  (wire (pts (xy 82.55 53.34) (xy 91.44 53.34))
+    (stroke (width 0) (type default) (color 0 0 0 0))
+  )
+  (wire (pts (xy 118.11 63.5) (xy 127 63.5))
+    (stroke (width 0) (type default) (color 0 0 0 0))
+  )
+  (wire (pts (xy 162.56 114.3) (xy 196.85 114.3))
+    (stroke (width 0) (type default) (color 0 0 0 0))
+  )
+  (wire (pts (xy 82.55 63.5) (xy 91.44 63.5))
+    (stroke (width 0) (type default) (color 0 0 0 0))
+  )
+  (wire (pts (xy 130.81 88.9) (xy 143.51 88.9))
+    (stroke (width 0) (type default) (color 0 0 0 0))
+  )
+  (wire (pts (xy 127 92.71) (xy 127 101.6))
+    (stroke (width 0) (type default) (color 0 0 0 0))
+  )
+  (wire (pts (xy 139.7 74.93) (xy 177.8 74.93))
+    (stroke (width 0) (type default) (color 0 0 0 0))
+  )
+  (wire (pts (xy 80.01 73.66) (xy 91.44 73.66))
+    (stroke (width 0) (type default) (color 0 0 0 0))
+  )
+  (wire (pts (xy 102.87 63.5) (xy 102.87 73.66))
+    (stroke (width 0) (type default) (color 0 0 0 0))
+  )
+  (wire (pts (xy 87.63 81.28) (xy 87.63 85.09))
+    (stroke (width 0) (type default) (color 0 0 0 0))
+  )
+  (wire (pts (xy 158.75 86.36) (xy 162.56 86.36))
+    (stroke (width 0) (type default) (color 0 0 0 0))
+  )
   (wire (pts (xy 177.8 86.36) (xy 196.85 86.36))
-    (stroke (width 0) (type default) (color 0 0 0 0))
-  )
-  (wire (pts (xy 127 76.2) (xy 121.92 76.2))
-    (stroke (width 0) (type default) (color 0 0 0 0))
-  )
-  (wire (pts (xy 130.81 88.9) (xy 143.51 88.9))
-    (stroke (width 0) (type default) (color 0 0 0 0))
-  )
-  (wire (pts (xy 127 76.2) (xy 127 85.09))
-    (stroke (width 0) (type default) (color 0 0 0 0))
-  )
-  (wire (pts (xy 102.87 73.66) (xy 106.68 73.66))
-    (stroke (width 0) (type default) (color 0 0 0 0))
-  )
-  (wire (pts (xy 177.8 86.36) (xy 173.99 86.36))
-    (stroke (width 0) (type default) (color 0 0 0 0))
-  )
-  (wire (pts (xy 177.8 86.36) (xy 177.8 90.17))
-    (stroke (width 0) (type default) (color 0 0 0 0))
-  )
-  (wire (pts (xy 83.82 81.28) (xy 87.63 81.28))
-    (stroke (width 0) (type default) (color 0 0 0 0))
-  )
-  (wire (pts (xy 177.8 74.93) (xy 177.8 86.36))
-    (stroke (width 0) (type default) (color 0 0 0 0))
-  )
-  (wire (pts (xy 162.56 86.36) (xy 166.37 86.36))
-    (stroke (width 0) (type default) (color 0 0 0 0))
-  )
-  (wire (pts (xy 76.2 81.28) (xy 72.39 81.28))
-    (stroke (width 0) (type default) (color 0 0 0 0))
-  )
-  (wire (pts (xy 72.39 77.47) (xy 72.39 81.28))
-    (stroke (width 0) (type default) (color 0 0 0 0))
-  )
-  (wire (pts (xy 110.49 63.5) (xy 102.87 63.5))
-    (stroke (width 0) (type default) (color 0 0 0 0))
-  )
-  (wire (pts (xy 99.06 63.5) (xy 102.87 63.5))
-    (stroke (width 0) (type default) (color 0 0 0 0))
-  )
-  (wire (pts (xy 102.87 53.34) (xy 102.87 63.5))
-    (stroke (width 0) (type default) (color 0 0 0 0))
-  )
-  (wire (pts (xy 82.55 53.34) (xy 91.44 53.34))
-    (stroke (width 0) (type default) (color 0 0 0 0))
-  )
-  (wire (pts (xy 118.11 63.5) (xy 127 63.5))
-    (stroke (width 0) (type default) (color 0 0 0 0))
-  )
-  (wire (pts (xy 162.56 114.3) (xy 196.85 114.3))
-    (stroke (width 0) (type default) (color 0 0 0 0))
-  )
-  (wire (pts (xy 82.55 63.5) (xy 91.44 63.5))
-    (stroke (width 0) (type default) (color 0 0 0 0))
-  )
-  (wire (pts (xy 127 92.71) (xy 127 101.6))
-    (stroke (width 0) (type default) (color 0 0 0 0))
-  )
-  (wire (pts (xy 139.7 74.93) (xy 177.8 74.93))
-    (stroke (width 0) (type default) (color 0 0 0 0))
-  )
-  (wire (pts (xy 80.01 73.66) (xy 91.44 73.66))
-    (stroke (width 0) (type default) (color 0 0 0 0))
-  )
-  (wire (pts (xy 102.87 63.5) (xy 102.87 73.66))
-    (stroke (width 0) (type default) (color 0 0 0 0))
-  )
-  (wire (pts (xy 87.63 81.28) (xy 87.63 85.09))
-    (stroke (width 0) (type default) (color 0 0 0 0))
-  )
-  (wire (pts (xy 158.75 86.36) (xy 162.56 86.36))
     (stroke (width 0) (type default) (color 0 0 0 0))
   )
@@
     (pin "2")
   )
-  (symbol (lib_id "Device:R_Potentiometer") (at 80.01 81.28 90) (unit 1)
+  (symbol (lib_id "Device:R_Potentiometer") (at 80.01 81.28 270) (mirror x) (unit 1)
     (in_bom yes) (on_board yes) (fields_autoplaced)
     (property "Reference" "RV1" (id 0) (at 80.01 84.4455 90))
     (property "Value" "1k-offset_adj" (id 1) (at 80.01 87.2206 90))
-    (property "Footprint" "Potentiometer_THT:Potentiometer_Bourns_3339P_Vertical_HandSoldering" (id 2) (at 80.01 81.28 0)
-      (effects (font (size 1.27 1.27)) hide)
-    )
+    (property "Footprint" "Potentiometer_THT:Potentiometer_Vishay_T73YP_Vertical" (id 2) (at 80.01 81.28 0)
+      (effects (font (size 1.27 1.27)) hide)
+    )

Commit message: finished ch06 and added appendix
Parts:
- removed R3: 100k, Resistor_THT:R_Axial_DIN0207_L6.3mm_D2.5mm_P10.16mm_Horizontal, symbol Device:R
- removed RV1: 1k-offset_adj, Potentiometer_THT:Potentiometer_Vishay_T73YP_Vertical, symbol Device:R_Potentiometer
Other:
- moved on the sheet: R1, R2
Changed lines of the file:
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@@
-    (stroke (width 0) (type default) (color 0 0 0 0))
-  )
-  (wire (pts (xy 83.82 81.28) (xy 87.63 81.28))
     (stroke (width 0) (type default) (color 0 0 0 0))
   )
@@
     (stroke (width 0) (type default) (color 0 0 0 0))
   )
-  (wire (pts (xy 76.2 81.28) (xy 72.39 81.28))
-    (stroke (width 0) (type default) (color 0 0 0 0))
-  )
-  (wire (pts (xy 72.39 77.47) (xy 72.39 81.28))
-    (stroke (width 0) (type default) (color 0 0 0 0))
-  )
   (wire (pts (xy 110.49 63.5) (xy 102.87 63.5))
     (stroke (width 0) (type default) (color 0 0 0 0))
   )
+  (wire (pts (xy 99.06 73.66) (xy 102.87 73.66))
+    (stroke (width 0) (type default) (color 0 0 0 0))
+  )
+  (wire (pts (xy 82.55 63.5) (xy 91.44 63.5))
+    (stroke (width 0) (type default) (color 0 0 0 0))
+  )
+  (wire (pts (xy 118.11 63.5) (xy 127 63.5))
+    (stroke (width 0) (type default) (color 0 0 0 0))
+  )
+  (wire (pts (xy 162.56 114.3) (xy 196.85 114.3))
+    (stroke (width 0) (type default) (color 0 0 0 0))
+  )
+  (wire (pts (xy 82.55 73.66) (xy 91.44 73.66))
+    (stroke (width 0) (type default) (color 0 0 0 0))
+  )
+  (wire (pts (xy 130.81 88.9) (xy 143.51 88.9))
+    (stroke (width 0) (type default) (color 0 0 0 0))
+  )
+  (wire (pts (xy 127 92.71) (xy 127 101.6))
+    (stroke (width 0) (type default) (color 0 0 0 0))
+  )
+  (wire (pts (xy 139.7 74.93) (xy 177.8 74.93))
+    (stroke (width 0) (type default) (color 0 0 0 0))
+  )
+  (wire (pts (xy 102.87 63.5) (xy 102.87 73.66))
+    (stroke (width 0) (type default) (color 0 0 0 0))
+  )
+  (wire (pts (xy 158.75 86.36) (xy 162.56 86.36))
+    (stroke (width 0) (type default) (color 0 0 0 0))
+  )
+  (wire (pts (xy 177.8 86.36) (xy 196.85 86.36))
+    (stroke (width 0) (type default) (color 0 0 0 0))
+  )
+  (wire (pts (xy 102.87 78.74) (xy 102.87 82.55))
+    (stroke (width 0) (type default) (color 0 0 0 0))
+  )
   (wire (pts (xy 99.06 63.5) (xy 102.87 63.5))
     (stroke (width 0) (type default) (color 0 0 0 0))
   )
-  (wire (pts (xy 102.87 53.34) (xy 102.87 63.5))
-    (stroke (width 0) (type default) (color 0 0 0 0))
-  )
-  (wire (pts (xy 82.55 53.34) (xy 91.44 53.34))
-    (stroke (width 0) (type default) (color 0 0 0 0))
-  )
-  (wire (pts (xy 118.11 63.5) (xy 127 63.5))
-    (stroke (width 0) (type default) (color 0 0 0 0))
-  )
-  (wire (pts (xy 162.56 114.3) (xy 196.85 114.3))
-    (stroke (width 0) (type default) (color 0 0 0 0))
-  )
-  (wire (pts (xy 82.55 63.5) (xy 91.44 63.5))
-    (stroke (width 0) (type default) (color 0 0 0 0))
-  )
-  (wire (pts (xy 130.81 88.9) (xy 143.51 88.9))
-    (stroke (width 0) (type default) (color 0 0 0 0))
-  )
-  (wire (pts (xy 127 92.71) (xy 127 101.6))
-    (stroke (width 0) (type default) (color 0 0 0 0))
-  )
-  (wire (pts (xy 139.7 74.93) (xy 177.8 74.93))
-    (stroke (width 0) (type default) (color 0 0 0 0))
-  )
-  (wire (pts (xy 80.01 73.66) (xy 91.44 73.66))
-    (stroke (width 0) (type default) (color 0 0 0 0))
-  )
-  (wire (pts (xy 102.87 63.5) (xy 102.87 73.66))
-    (stroke (width 0) (type default) (color 0 0 0 0))
-  )
-  (wire (pts (xy 87.63 81.28) (xy 87.63 85.09))
-    (stroke (width 0) (type default) (color 0 0 0 0))
-  )
-  (wire (pts (xy 158.75 86.36) (xy 162.56 86.36))
-    (stroke (width 0) (type default) (color 0 0 0 0))
-  )
-  (wire (pts (xy 177.8 86.36) (xy 196.85 86.36))
-    (stroke (width 0) (type default) (color 0 0 0 0))
-  )
-  (wire (pts (xy 80.01 73.66) (xy 80.01 77.47))
-    (stroke (width 0) (type default) (color 0 0 0 0))
-  )
-  (wire (pts (xy 102.87 78.74) (xy 102.87 82.55))
-    (stroke (width 0) (type default) (color 0 0 0 0))
-  )
-  (wire (pts (xy 99.06 53.34) (xy 102.87 53.34))
-    (stroke (width 0) (type default) (color 0 0 0 0))
-  )
   (wire (pts (xy 106.68 78.74) (xy 102.87 78.74))
     (stroke (width 0) (type default) (color 0 0 0 0))
@@
   )
   (wire (pts (xy 162.56 86.36) (xy 162.56 114.3))
-    (stroke (width 0) (type default) (color 0 0 0 0))
-  )
-  (wire (pts (xy 99.06 73.66) (xy 102.87 73.66))
     (stroke (width 0) (type default) (color 0 0 0 0))
   )
@@
     (effects (font (size 1.27 1.27)) (justify left))
   )
-  (hierarchical_label "Manual_mod" (shape input) (at 82.55 53.34 180)
+  (hierarchical_label "Manual_mod" (shape input) (at 82.55 63.5 180)
     (effects (font (size 1.27 1.27)) (justify right))
   )
-  (hierarchical_label "LFO_mod" (shape input) (at 82.55 63.5 180)
+  (hierarchical_label "LFO_mod" (shape input) (at 82.55 73.66 180)
     (effects (font (size 1.27 1.27)) (justify right))
   )
-  (symbol (lib_id "Device:R") (at 95.25 53.34 90) (unit 1)
-    (in_bom yes) (on_board yes) (fields_autoplaced)
-    (property "Reference" "R1" (id 0) (at 95.25 48.3575 90))
-    (property "Value" "100k" (id 1) (at 95.25 51.1326 90))
-    (property "Footprint" "Resistor_THT:R_Axial_DIN0207_L6.3mm_D2.5mm_P10.16mm_Horizontal" (id 2) (at 95.25 55.118 90)
-      (effects (font (size 1.27 1.27)) hide)
-    )
-    (property "Datasheet" "~" (id 3) (at 95.25 53.34 0)
+  (symbol (lib_id "Device:R") (at 95.25 63.5 90) (unit 1)
+    (in_bom yes) (on_board yes) (fields_autoplaced)
+    (property "Reference" "R1" (id 0) (at 95.25 58.5175 90))
+    (property "Value" "100k" (id 1) (at 95.25 61.2926 90))
+    (property "Footprint" "Resistor_THT:R_Axial_DIN0207_L6.3mm_D2.5mm_P10.16mm_Horizontal" (id 2) (at 95.25 65.278 90)
+      (effects (font (size 1.27 1.27)) hide)
+    )
+    (property "Datasheet" "~" (id 3) (at 95.25 63.5 0)
       (effects (font (size 1.27 1.27)) hide)
     )
@@
     (pin "2")
   )
-  (symbol (lib_id "power:+12V") (at 72.39 77.47 0) (unit 1)
-    (in_bom yes) (on_board yes) (fields_autoplaced)
-    (property "Reference" "#PWR0110" (id 0) (at 72.39 81.28 0)
-      (effects (font (size 1.27 1.27)) hide)
-    )
-    (property "Value" "+12V" (id 1) (at 72.39 73.8655 0))
-    (property "Footprint" "" (id 2) (at 72.39 77.47 0)
-      (effects (font (size 1.27 1.27)) hide)
-    )
-    (property "Datasheet" "" (id 3) (at 72.39 77.47 0)
-      (effects (font (size 1.27 1.27)) hide)
-    )
-    (pin "1")
-  )
   (symbol (lib_id "Amplifier_Operational:TL074") (at 114.3 76.2 0) (mirror x) (unit 4)
     (in_bom yes) (on_board yes) (fields_autoplaced)
@@
   (symbol (lib_id "Device:R") (at 95.25 73.66 90) (unit 1)
     (in_bom yes) (on_board yes) (fields_autoplaced)
-    (property "Reference" "R3" (id 0) (at 95.25 68.6775 90))
+    (property "Reference" "R2" (id 0) (at 95.25 68.6775 90))
     (property "Value" "100k" (id 1) (at 95.25 71.4526 90))
     (property "Footprint" "Resistor_THT:R_Axial_DIN0207_L6.3mm_D2.5mm_P10.16mm_Horizontal" (id 2) (at 95.25 75.438 90)
@@
     (pin "1")
     (pin "2")
-  )
-  (symbol (lib_id "Device:R") (at 95.25 63.5 90) (unit 1)
-    (in_bom yes) (on_board yes) (fields_autoplaced)
-    (property "Reference" "R2" (id 0) (at 95.25 58.5175 90))
-    (property "Value" "100k" (id 1) (at 95.25 61.2926 90))
-    (property "Footprint" "Resistor_THT:R_Axial_DIN0207_L6.3mm_D2.5mm_P10.16mm_Horizontal" (id 2) (at 95.25 65.278 90)
-      (effects (font (size 1.27 1.27)) hide)
-    )
-    (property "Datasheet" "~" (id 3) (at 95.25 63.5 0)
-      (effects (font (size 1.27 1.27)) hide)
-    )
-    (pin "1")
-    (pin "2")
-  )
-  (symbol (lib_id "power:GNDD") (at 87.63 85.09 0) (unit 1)
-    (in_bom yes) (on_board yes)
-    (property "Reference" "#PWR0109" (id 0) (at 87.63 91.44 0)
-      (effects (font (size 1.27 1.27)) hide)
-    )
-    (property "Value" "GNDD" (id 1) (at 87.63 89.2715 0))
-    (property "Footprint" "" (id 2) (at 87.63 85.09 0)
-      (effects (font (size 1.27 1.27)) hide)
-    )
-    (property "Datasheet" "" (id 3) (at 87.63 85.09 0)
-      (effects (font (size 1.27 1.27)) hide)
-    )
-    (pin "1")
   )
   (symbol (lib_id "power:GNDD") (at 127 101.6 0) (unit 1)
@@
     (pin "2")
   )
-  (symbol (lib_id "Device:R_Potentiometer") (at 80.01 81.28 270) (mirror x) (unit 1)
-    (in_bom yes) (on_board yes) (fields_autoplaced)
-    (property "Reference" "RV1" (id 0) (at 80.01 84.4455 90))
-    (property "Value" "1k-offset_adj" (id 1) (at 80.01 87.2206 90))
-    (property "Footprint" "Potentiometer_THT:Potentiometer_Vishay_T73YP_Vertical" (id 2) (at 80.01 81.28 0)
-      (effects (font (size 1.27 1.27)) hide)
-    )
-    (property "Datasheet" "~" (id 3) (at 80.01 81.28 0)
-      (effects (font (size 1.27 1.27)) hide)
-    )
-    (pin "1")
-    (pin "2")
-    (pin "3")
-  )
 )
