File: FG-VCO-(core1)/v_oct_conv.kicad_sch (KiCad schematic)
At the start: 9 parts, among them J6 Exponential Test, Q1 MPQ3904, U1 TL074

Commit message: finished ch06 and added appendix
Parts:
- added R?: 1k2, Resistor_THT:R_Axial_DIN0207_L6.3mm_D2.5mm_P10.16mm_Horizontal, symbol Device:R
- R6: value 2M2 -> 1M
- R7: value 3k9 -> 10k
Connections:
- net at C3.2, R7.2, U1.7: now also R?.2; no longer Q1.12
- new net: Q1.12, R?.1
Other:
- moved on the sheet: Q1D
Changed lines of the file:
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@@
     (stroke (width 0) (type default) (color 0 0 0 0))
   )
-  (wire (pts (xy 147.32 88.9) (xy 152.4 88.9))
+  (wire (pts (xy 147.32 85.09) (xy 152.4 85.09))
     (stroke (width 0) (type default) (color 0 0 0 0))
   )
@@
     (stroke (width 0) (type default) (color 0 0 0 0))
   )
-  (wire (pts (xy 139.7 93.98) (xy 139.7 102.87))
-    (stroke (width 0) (type default) (color 0 0 0 0))
-  )
   (wire (pts (xy 121.92 102.87) (xy 127 102.87))
     (stroke (width 0) (type default) (color 0 0 0 0))
@@
     (stroke (width 0) (type default) (color 0 0 0 0))
   )
-  (wire (pts (xy 152.4 71.12) (xy 152.4 88.9))
+  (wire (pts (xy 152.4 71.12) (xy 152.4 85.09))
     (stroke (width 0) (type default) (color 0 0 0 0))
   )
@@
     (stroke (width 0) (type default) (color 0 0 0 0))
   )
+  (wire (pts (xy 139.7 100.33) (xy 139.7 102.87))
+    (stroke (width 0) (type default) (color 0 0 0 0))
+  )
+  (wire (pts (xy 139.7 90.17) (xy 139.7 92.71))
+    (stroke (width 0) (type default) (color 0 0 0 0))
+  )
   (wire (pts (xy 127 85.09) (xy 127 102.87))
     (stroke (width 0) (type default) (color 0 0 0 0))
@@
     (stroke (width 0) (type default) (color 0 0 0 0))
   )
-  (wire (pts (xy 139.7 71.12) (xy 139.7 83.82))
+  (wire (pts (xy 139.7 71.12) (xy 139.7 80.01))
     (stroke (width 0) (type default) (color 0 0 0 0))
   )
@@
     )
     (pin "1")
+  )
+  (symbol (lib_id "Device:R") (at 139.7 96.52 0) (mirror y) (unit 1)
+    (in_bom yes) (on_board yes)
+    (property "Reference" "R?" (id 0) (at 141.605 95.25 0)
+      (effects (font (size 1.27 1.27)) (justify right))
+    )
+    (property "Value" "1k2" (id 1) (at 141.605 97.79 0)
+      (effects (font (size 1.27 1.27)) (justify right))
+    )
+    (property "Footprint" "Resistor_THT:R_Axial_DIN0207_L6.3mm_D2.5mm_P10.16mm_Horizontal" (id 2) (at 141.478 96.52 90)
+      (effects (font (size 1.27 1.27)) hide)
+    )
+    (property "Datasheet" "~" (id 3) (at 139.7 96.52 0)
+      (effects (font (size 1.27 1.27)) hide)
+    )
+    (pin "1")
+    (pin "2")
   )
   (symbol (lib_id "power:GNDD") (at 63.5 167.64 0) (unit 1)
@@
     (pin "1")
   )
-  (symbol (lib_id "Custom:MPQ3904") (at 139.7 88.9 0) (mirror y) (unit 4)
-    (in_bom yes) (on_board yes) (fields_autoplaced)
-    (property "Reference" "Q1" (id 0) (at 137.3886 87.9915 0)
-      (effects (font (size 1.27 1.27)) (justify left))
-    )
-    (property "Value" "MPQ3904" (id 1) (at 137.3886 90.7666 0)
-      (effects (font (size 1.27 1.27)) (justify left))
-    )
-    (property "Footprint" "Custom Footprints:DIP-14_central_caps" (id 2) (at 133.35 87.63 0)
-      (effects (font (size 1.27 1.27)) hide)
-    )
-    (property "Datasheet" "" (id 3) (at 133.35 87.63 0)
+  (symbol (lib_id "Custom:MPQ3904") (at 139.7 85.09 0) (mirror y) (unit 4)
+    (in_bom yes) (on_board yes) (fields_autoplaced)
+    (property "Reference" "Q1" (id 0) (at 137.3886 84.1815 0)
+      (effects (font (size 1.27 1.27)) (justify left))
+    )
+    (property "Value" "MPQ3904" (id 1) (at 137.3886 86.9566 0)
+      (effects (font (size 1.27 1.27)) (justify left))
+    )
+    (property "Footprint" "Custom Footprints:DIP-14_central_caps" (id 2) (at 133.35 83.82 0)
+      (effects (font (size 1.27 1.27)) hide)
+    )
+    (property "Datasheet" "" (id 3) (at 133.35 83.82 0)
       (effects (font (size 1.27 1.27)) hide)
     )
@@
       (effects (font (size 1.27 1.27)) (justify right))
     )
-    (property "Value" "3k9" (id 1) (at 121.92 78.74 0)
+    (property "Value" "10k" (id 1) (at 121.92 78.74 0)
       (effects (font (size 1.27 1.27)) (justify right))
     )
@@
       (effects (font (size 1.27 1.27)) (justify left))
     )
-    (property "Value" "2M2" (id 1) (at 128.778 51.3966 0)
-      (effects (font (size 1.27 1.27)) (justify left))
-    )
+    (property "Value" "1M" (id 1) (at 128.778 51.3966 0)
+      (effects (font (size 1.27 1.27)) (justify left))
+    )
