File: FG-VCO-(core2)/ffs.kicad_sch (KiCad schematic)
At the start: 2 parts, among them U1 74LS73

Commit message: same as previous, for the whole folder
Connections:
- net +5V: now also U1.14 (J), U1.3 (K); no longer U1.10 (K), U1.7 (J)
- net RCO: now also U1.10 (K), U1.7 (J); no longer U1.14 (J), U1.3 (K)
- net U/D: now also U1.9 (Q); no longer U1.12 (Q)
- net f_clk/2: now also U1.12 (Q); no longer U1.9 (Q)
Other:
- moved on the sheet: U1A, U1B
Changed lines of the file:
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@@
     (pin "1")
   )
-  (symbol (lib_id "74xx:74LS73") (at 107.95 107.95 0) (mirror x) (unit 1)
+  (symbol (lib_id "74xx:74LS73") (at 107.95 69.85 0) (mirror x) (unit 1)
     (in_bom yes) (on_board yes) (fields_autoplaced)
-    (property "Reference" "U1" (id 0) (at 107.95 116.9965 0))
-    (property "Value" "74LS73" (id 1) (at 107.95 114.2214 0))
-    (property "Footprint" "Custom Footprints:DIP-14_central_caps" (id 2) (at 107.95 107.95 0)
+    (property "Reference" "U1" (id 0) (at 107.95 78.8965 0))
+    (property "Value" "74LS73" (id 1) (at 107.95 76.1214 0))
+    (property "Footprint" "Custom Footprints:DIP-14_central_caps" (id 2) (at 107.95 69.85 0)
       (effects (font (size 1.27 1.27)) hide)
     )
-    (property "Datasheet" "http://www.ti.com/lit/gpn/sn74LS73" (id 3) (at 107.95 107.95 0)
+    (property "Datasheet" "http://www.ti.com/lit/gpn/sn74LS73" (id 3) (at 107.95 69.85 0)
       (effects (font (size 1.27 1.27)) hide)
     )
@@
     (pin "9")
   )
-  (symbol (lib_id "74xx:74LS73") (at 107.95 69.85 0) (mirror x) (unit 2)
+  (symbol (lib_id "74xx:74LS73") (at 107.95 107.95 0) (mirror x) (unit 2)
     (in_bom yes) (on_board yes) (fields_autoplaced)
-    (property "Reference" "U1" (id 0) (at 107.95 77.0795 0))
-    (property "Value" "74LS73" (id 1) (at 107.95 79.8546 0))
-    (property "Footprint" "Custom Footprints:DIP-14_central_caps" (id 2) (at 107.95 69.85 0)
+    (property "Reference" "U1" (id 0) (at 107.95 115.1795 0))
+    (property "Value" "74LS73" (id 1) (at 107.95 117.9546 0))
+    (property "Footprint" "Custom Footprints:DIP-14_central_caps" (id 2) (at 107.95 107.95 0)
       (effects (font (size 1.27 1.27)) hide)
     )
-    (property "Datasheet" "http://www.ti.com/lit/gpn/sn74LS73" (id 3) (at 107.95 69.85 0)
+    (property "Datasheet" "http://www.ti.com/lit/gpn/sn74LS73" (id 3) (at 107.95 107.95 0)
       (effects (font (size 1.27 1.27)) hide)
     )

Commit message: finished ch06 and added appendix
Other:
- company: (none) -> Gottardo Filippo
- title: (none) -> FGVCO - Core 2
Changed lines of the file:
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@@
 (kicad_sch (version 20211123) (generator eeschema)
   (paper "A4")
+  (title_block
+    (title "FGVCO - Core 2")
+    (date "2022-05-31")
+    (company "Gottardo Filippo")
+  )
   (junction (at 95.25 82.55) (diameter 0) (color 0 0 0 0)
   )
