File: FG-VCO-(core2)/ramp_cntr.kicad_sch (KiCad schematic)
At the start: 2 parts, among them U8 74HC590

Commit message: finished ch06 and added appendix
Other:
- company: (none) -> Gottardo Filippo
- title: (none) -> FGVCO - Core 2
Changed lines of the file:
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@@
 (kicad_sch (version 20211123) (generator eeschema)
   (paper "A4")
+  (title_block
+    (title "FGVCO - Core 2")
+    (date "2022-05-31")
+    (company "Gottardo Filippo")
+  )
   (junction (at 120.65 95.25) (diameter 0) (color 0 0 0 0)
   )
