File: FG-VCO-(core2)/ramp_inverter.kicad_sch (KiCad schematic)
At the start: 4 parts, among them J11 Test Saw, U3 TL074

Commit message: same as previous, for the whole folder
Parts:
- removed U3: TL074, Custom Footprints:DIP-14_central_caps, symbol Amplifier_Operational:TL074
- added U3: TL082, Custom Footprints:DIP-8_central_caps, symbol Amplifier_Operational:TL082
Connections:
- net GNDD: now also U3.3 (+)
- net V_saw: now also U3.1
- net at R25.2, R26.1: now also U3.2 (-)
Changed lines of the file:
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@@
     (effects (font (size 1.27 1.27)) (justify left))
-  )
-  (symbol (lib_id "Amplifier_Operational:TL074") (at 133.35 69.85 0) (mirror x) (unit 3)
-    (in_bom yes) (on_board yes) (fields_autoplaced)
-    (property "Reference" "U3" (id 0) (at 133.35 60.8035 0))
-    (property "Value" "TL074" (id 1) (at 133.35 63.5786 0))
-    (property "Footprint" "Custom Footprints:DIP-14_central_caps" (id 2) (at 132.08 72.39 0)
-      (effects (font (size 1.27 1.27)) hide)
-    )
-    (property "Datasheet" "http://www.ti.com/lit/ds/symlink/tl071.pdf" (id 3) (at 134.62 74.93 0)
-      (effects (font (size 1.27 1.27)) hide)
-    )
-    (pin "10")
-    (pin "8")
-    (pin "9")
   )
   (symbol (lib_id "power:GNDD") (at 123.19 74.93 0) (unit 1)
@@
     (pin "2")
   )
+  (symbol (lib_id "Amplifier_Operational:TL082") (at 133.35 69.85 0) (mirror x) (unit 1)
+    (in_bom yes) (on_board yes) (fields_autoplaced)
+    (property "Reference" "U3" (id 0) (at 133.35 60.8035 0))
+    (property "Value" "TL082" (id 1) (at 133.35 63.5786 0))
+    (property "Footprint" "Custom Footprints:DIP-8_central_caps" (id 2) (at 133.35 69.85 0)
+      (effects (font (size 1.27 1.27)) hide)
+    )
+    (property "Datasheet" "http://www.ti.com/lit/ds/symlink/tl081.pdf" (id 3) (at 133.35 69.85 0)
+      (effects (font (size 1.27 1.27)) hide)
+    )
+    (pin "1")
+    (pin "2")
+    (pin "3")
+  )
   (symbol (lib_id "Device:R") (at 116.84 67.31 90) (unit 1)

Commit message: finished ch06 and added appendix
Other:
- company: (none) -> Gottardo Filippo
- title: (none) -> FGVCO - Core 2
Changed lines of the file:
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@@
 (kicad_sch (version 20211123) (generator eeschema)
   (paper "A4")
+  (title_block
+    (title "FGVCO - Core 2")
+    (date "2022-05-31")
+    (company "Gottardo Filippo")
+  )
   (junction (at 143.51 69.85) (diameter 0) (color 0 0 0 0)
   )
