File: FG-VCO-(core2)/square_adapter.kicad_sch (KiCad schematic)
At the start: 4 parts, among them J7 Test Square, U3 TL074

Commit message: same as previous, for the whole folder
Parts:
- removed U3: TL074, Custom Footprints:DIP-14_central_caps, symbol Amplifier_Operational:TL074
- added U3: TL082, Custom Footprints:DIP-8_central_caps, symbol Amplifier_Operational:TL082
Connections:
- net V_square: now also U3.7
- net at RV2.2: now also U3.5 (+)
- net at RV3.2: now also U3.6 (-)
Changed lines of the file:
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@@
-    (stroke (width 0) (type default) (color 0 0 0 0))
-  )
-  (wire (pts (xy 135.89 73.66) (xy 135.89 80.01))
     (stroke (width 0) (type default) (color 0 0 0 0))
   )
@@
   )
   (wire (pts (xy 153.67 82.55) (xy 156.21 82.55))
+    (stroke (width 0) (type default) (color 0 0 0 0))
+  )
+  (wire (pts (xy 135.89 73.66) (xy 135.89 80.01))
     (stroke (width 0) (type default) (color 0 0 0 0))
   )
@@
     (pin "3")
   )
-  (symbol (lib_id "Amplifier_Operational:TL074") (at 146.05 82.55 0) (mirror x) (unit 4)
+  (symbol (lib_id "Amplifier_Operational:TL082") (at 146.05 82.55 0) (mirror x) (unit 2)
     (in_bom yes) (on_board yes) (fields_autoplaced)
     (property "Reference" "U3" (id 0) (at 146.05 73.5035 0))
-    (property "Value" "TL074" (id 1) (at 146.05 76.2786 0))
-    (property "Footprint" "Custom Footprints:DIP-14_central_caps" (id 2) (at 144.78 85.09 0)
+    (property "Value" "TL082" (id 1) (at 146.05 76.2786 0))
+    (property "Footprint" "Custom Footprints:DIP-8_central_caps" (id 2) (at 146.05 82.55 0)
       (effects (font (size 1.27 1.27)) hide)
     )
-    (property "Datasheet" "http://www.ti.com/lit/ds/symlink/tl071.pdf" (id 3) (at 147.32 87.63 0)
+    (property "Datasheet" "http://www.ti.com/lit/ds/symlink/tl081.pdf" (id 3) (at 146.05 82.55 0)
       (effects (font (size 1.27 1.27)) hide)
     )
-    (pin "12")
-    (pin "13")
-    (pin "14")
+    (pin "5")
+    (pin "6")
+    (pin "7")
   )
   (symbol (lib_id "power:+5V") (at 107.95 88.9 0) (unit 1)

Commit message: finished ch06 and added appendix
Other:
- company: (none) -> Gottardo Filippo
- title: (none) -> FGVCO - Core 2
Changed lines of the file:
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@@
 (kicad_sch (version 20211123) (generator eeschema)
   (paper "A4")
+  (title_block
+    (title "FGVCO - Core 2")
+    (date "2022-05-31")
+    (company "Gottardo Filippo")
+  )
   (junction (at 156.21 82.55) (diameter 0) (color 0 0 0 0)
   )
