File: FG-VCO-(core2)/triangle_cntr.kicad_sch (KiCad schematic)
At the start: 7 parts, among them Q2 2N7000, U10 74LS169, U11 74LS169

Commit message: finished ch06 and added appendix
Other:
- company: (none) -> Gottardo Filippo
- title: (none) -> FGVCO - Core 2
Changed lines of the file:
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@@
 (kicad_sch (version 20211123) (generator eeschema)
   (paper "A4")
+  (title_block
+    (title "FGVCO - Core 2")
+    (date "2022-05-31")
+    (company "Gottardo Filippo")
+  )
   (junction (at 114.3 107.95) (diameter 0) (color 0 0 0 0)
   )
