File: FG-VCO-(core2)/FG-VCO-(core2).kicad_sch (KiCad schematic)
At the start: 14 parts, among them J1 main_power, J14 conn_power, J2 conn_signals_1, J3 conn_signals_2, J8 conn_signals_3, U3 TL074, U4 TL082

Commit message: same as previous, for the whole folder
Parts:
- removed U3: TL074, Custom Footprints:DIP-14_central_caps, symbol Amplifier_Operational:TL074
- added U3: TL082, Custom Footprints:DIP-8_central_caps, symbol Amplifier_Operational:TL082
Connections:
- net +12V: now also U3.8 (V+)
- net -12V: now also U3.4 (V-)
Changed lines of the file:
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@@
     (pin "1")
-  )
-  (symbol (lib_id "Amplifier_Operational:TL074") (at 173.99 139.7 0) (unit 5)
-    (in_bom yes) (on_board yes) (fields_autoplaced)
-    (property "Reference" "U3" (id 0) (at 172.085 138.7915 0)
-      (effects (font (size 1.27 1.27)) (justify left))
-    )
-    (property "Value" "TL074" (id 1) (at 172.085 141.5666 0)
-      (effects (font (size 1.27 1.27)) (justify left))
-    )
-    (property "Footprint" "Custom Footprints:DIP-14_central_caps" (id 2) (at 172.72 137.16 0)
-      (effects (font (size 1.27 1.27)) hide)
-    )
-    (property "Datasheet" "http://www.ti.com/lit/ds/symlink/tl071.pdf" (id 3) (at 175.26 134.62 0)
-      (effects (font (size 1.27 1.27)) hide)
-    )
-    (pin "11")
-    (pin "4")
   )
   (symbol (lib_id "Mechanical:MountingHole") (at 260.35 128.27 0) (unit 1)
@@
       (effects (font (size 1.27 1.27)) hide)
     )
+  )
+  (symbol (lib_id "Amplifier_Operational:TL082") (at 173.99 139.7 0) (unit 3)
+    (in_bom yes) (on_board yes) (fields_autoplaced)
+    (property "Reference" "U3" (id 0) (at 172.085 138.7915 0)
+      (effects (font (size 1.27 1.27)) (justify left))
+    )
+    (property "Value" "TL082" (id 1) (at 172.085 141.5666 0)
+      (effects (font (size 1.27 1.27)) (justify left))
+    )
+    (property "Footprint" "Custom Footprints:DIP-8_central_caps" (id 2) (at 173.99 139.7 0)
+      (effects (font (size 1.27 1.27)) hide)
+    )
+    (property "Datasheet" "http://www.ti.com/lit/ds/symlink/tl081.pdf" (id 3) (at 173.99 139.7 0)
+      (effects (font (size 1.27 1.27)) hide)
+    )
+    (pin "4")
+    (pin "8")
   )
   (symbol (lib_id "power:GNDD") (at 152.4 142.24 0) (unit 1)
@@
   )
   (symbol_instances
+    (path "/816eded2-4d1e-4711-b80f-520d0bcc8084/8a7a9492-ab89-4516-a214-7040d82b61b8"
+      (reference "#PWR01") (unit 1) (value "+12V") (footprint "")
+    )
+    (path "/816eded2-4d1e-4711-b80f-520d0bcc8084/0c90f154-42bc-421b-9657-49ed475a766c"
+      (reference "#PWR02") (unit 1) (value "-12V") (footprint "")
+    )
     (path "/5367af2e-e61d-4c69-b2db-1b855ecafab9"
       (reference "#PWR03") (unit 1) (value "+12V") (footprint "")
@@
       (reference "#PWR010") (unit 1) (value "GNDD") (footprint "")
     )
+    (path "/816eded2-4d1e-4711-b80f-520d0bcc8084/54d1bef2-3394-413b-aee9-ac2cc465686b"
+      (reference "#PWR011") (unit 1) (value "GNDD") (footprint "")
+    )
     (path "/b86fe704-c129-4192-a47d-bc6810198c37"
       (reference "#PWR014") (unit 1) (value "+5V") (footprint "")
@@
       (reference "C5") (unit 1) (value "4n7") (footprint "Custom Footprints:C_Disc_P2.54mm")
     )
+    (path "/816eded2-4d1e-4711-b80f-520d0bcc8084/c2e1af5c-e691-45b2-ba84-605035166d14"
+      (reference "C6") (unit 1) (value "4n7") (footprint "Custom Footprints:C_Disc_P2.54mm")
+    )
+    (path "/816eded2-4d1e-4711-b80f-520d0bcc8084/4977eead-85b2-4898-97b1-0686002855f4"
+      (reference "C7") (unit 1) (value "4n7") (footprint "Custom Footprints:C_Disc_P2.54mm")
+    )
     (path "/8722e585-87bf-491c-9cc4-42f8ede200d3/d363207b-14eb-4bc8-ab06-2b29f12946b6"
       (reference "C15") (unit 1) (value "100n") (footprint "Custom Footprints:C_Disc_P2.54mm")
@@
       (reference "U1") (unit 3) (value "74LS73") (footprint "Custom Footprints:DIP-14_central_caps")
     )
-    (path "/816eded2-4d1e-4711-b80f-520d0bcc8084/f9d3f3a2-be5e-4fb5-b3b0-0fdf1fa8bc0c"
-      (reference "U3") (unit 1) (value "TL074") (footprint "Custom Footprints:DIP-14_central_caps")
-    )
-    (path "/816eded2-4d1e-4711-b80f-520d0bcc8084/0676be3b-4ef5-468b-97b5-f6cf2caec143"
-      (reference "U3") (unit 2) (value "TL074") (footprint "Custom Footprints:DIP-14_central_caps")
-    )
-    (path "/32893f07-87d9-4ecf-894a-bda4253ed38d/23481648-802a-4acb-ba60-96be3681d37d"
-      (reference "U3") (unit 3) (value "TL074") (footprint "Custom Footprints:DIP-14_central_caps")
-    )
-    (path "/6e243853-c636-475f-a906-22f4eb43cb8e/41009f2b-b7b8-4c73-a957-bddea2557205"
-      (reference "U3") (unit 4) (value "TL074") (footprint "Custom Footprints:DIP-14_central_caps")
-    )
-    (path "/e1e89ebc-d05f-4d57-9fe1-5715a85d7766"
-      (reference "U3") (unit 5) (value "TL074") (footprint "Custom Footprints:DIP-14_central_caps")
+    (path "/816eded2-4d1e-4711-b80f-520d0bcc8084/caab9318-b634-42d4-8f60-25e2241c571e"
+      (reference "U2") (unit 1) (value "TL082") (footprint "Custom Footprints:DIP-8_central_caps")
+    )
+    (path "/816eded2-4d1e-4711-b80f-520d0bcc8084/f58c3928-37aa-4b6c-bc79-caa7d95369b8"
+      (reference "U2") (unit 2) (value "TL082") (footprint "Custom Footprints:DIP-8_central_caps")
+    )
+    (path "/816eded2-4d1e-4711-b80f-520d0bcc8084/23fe10f6-009e-409d-9387-bdfb557102be"
+      (reference "U2") (unit 3) (value "TL082") (footprint "Custom Footprints:DIP-8_central_caps")
+    )
+    (path "/32893f07-87d9-4ecf-894a-bda4253ed38d/f580492c-4129-4e47-be22-b6d42d63748b"
+      (reference "U3") (unit 1) (value "TL082") (footprint "Custom Footprints:DIP-8_central_caps")
+    )
+    (path "/6e243853-c636-475f-a906-22f4eb43cb8e/4c1a79f0-6b5d-45e4-8e71-196f0d87c8d2"
+      (reference "U3") (unit 2) (value "TL082") (footprint "Custom Footprints:DIP-8_central_caps")
+    )
+    (path "/e6fb3009-f959-44f3-9992-a3165a8cefe3"
+      (reference "U3") (unit 3) (value "TL082") (footprint "Custom Footprints:DIP-8_central_caps")
     )
     (path "/cdef380b-324f-46f1-b1d1-a124b95f8ef4/1784be64-8efd-4f48-b3cd-98719258b9ca"

Commit message: finished ch06 and added appendix
Other:
- title: FGVCO -> FGVCO - Core 2
Changed lines of the file:
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@@
   (paper "A4")
   (title_block
-    (title "FGVCO")
+    (title "FGVCO - Core 2")
     (date "2022-05-31")
     (rev "0")
