File: FG-VCO-(core2)/tri_sin_conv.kicad_sch (KiCad schematic)
At the start: 11 parts, among them J6 Test Sine, U3 TL074

Commit message: same as previous, for the whole folder
Parts:
- removed U3: TL074, Custom Footprints:DIP-14_central_caps, symbol Amplifier_Operational:TL074
- added C6, C7: 4n7, Custom Footprints:C_Disc_P2.54mm, symbol Device:C
- added U2: TL082, Custom Footprints:DIP-8_central_caps, symbol Amplifier_Operational:TL082
Connections:
- net GNDD: now also C6.2, C7.1, U2.3 (+)
- net V_sine: now also U2.7
- net at D2.1 (K), D3.1 (K), D4.2 (A)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: now also U2.1, U2.5 (+)
- net at R17.2, R18.1: now also U2.6 (-)
- net at D1.1 (K), R14.2, R15.1: now also U2.2 (-)
- new net +12V: C6.1, U2.8 (V+)
- new net -12V: C7.2, U2.4 (V-)

Commit message: finished ch06 and added appendix
Other:
- company: (none) -> Gottardo Filippo
- title: (none) -> FGVCO - Core 2
Changed lines of the file:
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@@
 (kicad_sch (version 20211123) (generator eeschema)
   (paper "A4")
+  (title_block
+    (title "FGVCO - Core 2")
+    (date "2022-05-31")
+    (company "Gottardo Filippo")
+  )
   (junction (at 124.46 60.96) (diameter 0) (color 0 0 0 0)
   )

Commit message: completed
Parts:
- removed R17: 22k, Resistor_THT:R_Axial_DIN0207_L6.3mm_D2.5mm_P10.16mm_Horizontal, symbol Device:R
- removed R18: 33k, Resistor_THT:R_Axial_DIN0207_L6.3mm_D2.5mm_P10.16mm_Horizontal, symbol Device:R
- added RV1: 50k - gain, symbol Device:R_Potentiometer
- R14: value 10k -> 33k
- R15: value 10k -> 22k
- R16: value 22k -> 12k
Connections:
- net GNDD: now also RV1.1
- net V_sine: now also RV1.3
- net at U2.6 (-): now also RV1.2
Changed lines of the file:
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@@
   (junction (at 124.46 73.66) (diameter 0) (color 0 0 0 0)
   )
-  (junction (at 168.91 105.41) (diameter 0) (color 0 0 0 0)
-  )
   (junction (at 111.76 73.66) (diameter 0) (color 0 0 0 0)
   )
@@
     (stroke (width 0) (type default) (color 0 0 0 0))
   )
+  (wire (pts (xy 148.59 105.41) (xy 165.1 105.41))
+    (stroke (width 0) (type default) (color 0 0 0 0))
+  )
   (wire (pts (xy 121.92 73.66) (xy 124.46 73.66))
     (stroke (width 0) (type default) (color 0 0 0 0))
@@
     (stroke (width 0) (type default) (color 0 0 0 0))
   )
-  (wire (pts (xy 168.91 88.9) (xy 168.91 95.25))
+  (wire (pts (xy 168.91 88.9) (xy 168.91 101.6))
     (stroke (width 0) (type default) (color 0 0 0 0))
   )
@@
     (stroke (width 0) (type default) (color 0 0 0 0))
   )
-  (wire (pts (xy 168.91 115.57) (xy 168.91 121.92))
+  (wire (pts (xy 168.91 109.22) (xy 168.91 121.285))
     (stroke (width 0) (type default) (color 0 0 0 0))
   )
@@
     (stroke (width 0) (type default) (color 0 0 0 0))
   )
-  (wire (pts (xy 168.91 102.87) (xy 168.91 105.41))
-    (stroke (width 0) (type default) (color 0 0 0 0))
-  )
   (wire (pts (xy 134.62 35.56) (xy 137.16 35.56))
     (stroke (width 0) (type default) (color 0 0 0 0))
@@
     (stroke (width 0) (type default) (color 0 0 0 0))
   )
-  (wire (pts (xy 148.59 105.41) (xy 168.91 105.41))
-    (stroke (width 0) (type default) (color 0 0 0 0))
-  )
   (wire (pts (xy 134.62 73.66) (xy 137.16 73.66))
     (stroke (width 0) (type default) (color 0 0 0 0))
   )
   (wire (pts (xy 266.7 35.56) (xy 266.7 39.37))
-    (stroke (width 0) (type default) (color 0 0 0 0))
-  )
-  (wire (pts (xy 168.91 105.41) (xy 168.91 107.95))
     (stroke (width 0) (type default) (color 0 0 0 0))
   )
@@
     (effects (font (size 1.27 1.27)) (justify left))
   )
-  (symbol (lib_id "Device:R") (at 168.91 99.06 0) (unit 1)
-    (in_bom yes) (on_board yes) (fields_autoplaced)
-    (property "Reference" "R17" (id 0) (at 170.688 98.1515 0)
-      (effects (font (size 1.27 1.27)) (justify left))
-    )
-    (property "Value" "22k" (id 1) (at 170.688 100.9266 0)
-      (effects (font (size 1.27 1.27)) (justify left))
-    )
-    (property "Footprint" "Resistor_THT:R_Axial_DIN0207_L6.3mm_D2.5mm_P10.16mm_Horizontal" (id 2) (at 167.132 99.06 90)
-      (effects (font (size 1.27 1.27)) hide)
-    )
-    (property "Datasheet" "~" (id 3) (at 168.91 99.06 0)
-      (effects (font (size 1.27 1.27)) hide)
-    )
-    (pin "1")
-    (pin "2")
-  )
   (symbol (lib_id "power:-12V") (at 254 55.88 180) (unit 1)
     (in_bom yes) (on_board yes) (fields_autoplaced)
@@
     (in_bom yes) (on_board yes) (fields_autoplaced)
     (property "Reference" "R14" (id 0) (at 105.41 78.8375 90))
-    (property "Value" "10k" (id 1) (at 105.41 81.6126 90))
+    (property "Value" "33k" (id 1) (at 105.41 81.6126 90))
     (property "Footprint" "Resistor_THT:R_Axial_DIN0207_L6.3mm_D2.5mm_P10.16mm_Horizontal" (id 2) (at 105.41 85.598 90)
       (effects (font (size 1.27 1.27)) hide)
@@
     (pin "8")
   )
-  (symbol (lib_id "Device:R") (at 168.91 111.76 0) (unit 1)
-    (in_bom yes) (on_board yes) (fields_autoplaced)
-    (property "Reference" "R18" (id 0) (at 170.688 110.8515 0)
-      (effects (font (size 1.27 1.27)) (justify left))
-    )
-    (property "Value" "33k" (id 1) (at 170.688 113.6266 0)
-      (effects (font (size 1.27 1.27)) (justify left))
-    )
-    (property "Footprint" "Resistor_THT:R_Axial_DIN0207_L6.3mm_D2.5mm_P10.16mm_Horizontal" (id 2) (at 167.132 111.76 90)
-      (effects (font (size 1.27 1.27)) hide)
-    )
-    (property "Datasheet" "~" (id 3) (at 168.91 111.76 0)
-      (effects (font (size 1.27 1.27)) hide)
-    )
-    (pin "1")
-    (pin "2")
-  )
   (symbol (lib_id "Device:R") (at 130.81 73.66 90) (unit 1)
     (in_bom yes) (on_board yes) (fields_autoplaced)
     (property "Reference" "R16" (id 0) (at 130.81 68.6775 90))
-    (property "Value" "22k" (id 1) (at 130.81 71.4526 90))
+    (property "Value" "12k" (id 1) (at 130.81 71.4526 90))
     (property "Footprint" "Resistor_THT:R_Axial_DIN0207_L6.3mm_D2.5mm_P10.16mm_Horizontal" (id 2) (at 130.81 75.438 90)
       (effects (font (size 1.27 1.27)) hide)
@@
     (pin "1")
   )
+  (symbol (lib_id "Device:R_Potentiometer") (at 168.91 105.41 180) (unit 1)
+    (in_bom yes) (on_board yes) (fields_autoplaced)
+    (property "Reference" "RV1" (id 0) (at 170.688 104.5015 0)
+      (effects (font (size 1.27 1.27)) (justify right))
+    )
+    (property "Value" "50k - gain" (id 1) (at 170.688 107.2766 0)
+      (effects (font (size 1.27 1.27)) (justify right))
+    )
+    (property "Footprint" "" (id 2) (at 168.91 105.41 0)
+      (effects (font (size 1.27 1.27)) hide)
+    )
+    (property "Datasheet" "~" (id 3) (at 168.91 105.41 0)
+      (effects (font (size 1.27 1.27)) hide)
+    )
+    (pin "1")
+    (pin "2")
+    (pin "3")
+  )
   (symbol (lib_id "power:+12V") (at 254 22.86 0) (unit 1)
     (in_bom yes) (on_board yes) (fields_autoplaced)
@@
     (in_bom yes) (on_board yes) (fields_autoplaced)
     (property "Reference" "R15" (id 0) (at 118.11 68.6775 90))
-    (property "Value" "10k" (id 1) (at 118.11 71.4526 90))
+    (property "Value" "22k" (id 1) (at 118.11 71.4526 90))
     (property "Footprint" "Resistor_THT:R_Axial_DIN0207_L6.3mm_D2.5mm_P10.16mm_Horizontal" (id 2) (at 118.11 75.438 90)
       (effects (font (size 1.27 1.27)) hide)
@@
     (pin "2")
   )
-  (symbol (lib_id "power:GNDD") (at 168.91 121.92 0) (unit 1)
-    (in_bom yes) (on_board yes) (fields_autoplaced)
-    (property "Reference" "#PWR067" (id 0) (at 168.91 128.27 0)
-      (effects (font (size 1.27 1.27)) hide)
-    )
-    (property "Value" "GNDD" (id 1) (at 168.91 126.1015 0))
-    (property "Footprint" "" (id 2) (at 168.91 121.92 0)
-      (effects (font (size 1.27 1.27)) hide)
-    )
-    (property "Datasheet" "" (id 3) (at 168.91 121.92 0)
-      (effects (font (size 1.27 1.27)) hide)
-    )
+  (symbol (lib_id "power:GNDD") (at 168.91 121.285 0) (unit 1)
+    (in_bom yes) (on_board yes) (fields_autoplaced)
+    (property "Reference" "#PWR067" (id 0) (at 168.91 127.635 0)
+      (effects (font (size 1.27 1.27)) hide)
+    )
+    (property "Value" "GNDD" (id 1) (at 168.91 125.4665 0))
+    (property "Footprint" "" (id 2) (at 168.91 121.285 0)
+      (effects (font (size 1.27 1.27)) hide)
+    )
+    (property "Datasheet" "" (id 3) (at 168.91 121.285 0)
+      (effects (font (size 1.27 1.27)) hide)
+    )
