File: FG-VCO-(interface)/FG-VCO-(interface).kicad_pcb (KiCad board)
At the start: 2 copper layers, 53.3 x 106.7 mm, 38 parts, among them J1 Out 1, J10 conn_modulation, J11 gnd, J12 gnd, J13 conn_mode, J2 Out 2, J3 Out 3, J4 Out 4, J5 Out 5, J6 Pulse Out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

Commit message: same as previous, for the whole folder
Parts:
- added R10: 10k, Resistor_THT:R_Axial_DIN0207_L6.3mm_D2.5mm_P10.16mm_Horizontal, F.Cu at (20.3, 24.8)
- added R11: 100k, Resistor_THT:R_Axial_DIN0207_L6.3mm_D2.5mm_P10.16mm_Horizontal, F.Cu at (20.3, 31.1)
- RV7: value 1k-Fine -> 10k-Fine
Connections:
- RV6 pad 2: Manual_mod -> Net-(RV6-Pad2)
- RV6 pad 3: Net-(RV6-Pad3) -> -12V
- RV7 pad 1: Net-(RV6-Pad3) -> +12V
- RV7 pad 2: Net-(RV6-Pad3) -> Net-(RV7-Pad2)
Routing:
- net +12V: track 40.9 -> 70.8 mm
- net Net-(RV6-Pad3): track 29.8 -> 0.00 mm
- net Net-(RV7-Pad2): track 0.00 -> 18.5 mm
- net Net-(RV6-Pad2): track 0.00 -> 18.5 mm
- net Manual_mod: track 11.3 -> 25.3 mm
- net -12V: track 42.0 -> 50.2 mm
Other:
- outline, holes or cut-outs redrawn
