File: FG-VCO-(interface)/FG-VCO-(interface).kicad_sch (KiCad schematic)
At the start: 38 parts, among them J1 Out 1, J10 conn_modulation, J11 gnd, J12 gnd, J13 conn_mode, J2 Out 2, J3 Out 3, J4 Out 4, J5 Out 5, J6 Pulse Out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

Commit message: same as previous, for the whole folder
Parts:
- added R10: 10k, Resistor_THT:R_Axial_DIN0207_L6.3mm_D2.5mm_P10.16mm_Horizontal, symbol Device:R
- added R11: 100k, Resistor_THT:R_Axial_DIN0207_L6.3mm_D2.5mm_P10.16mm_Horizontal, symbol Device:R
- RV7: value 1k-Fine -> 10k-Fine
Connections:
- net +12V: now also RV7.1
- net -12V: now also RV6.3
- net Manual_mod: now also R10.2, R11.2; no longer RV6.2
- new net: R10.1, RV6.2
- new net: R11.1, RV7.2
Other:
- moved on the sheet: RV7
Changed lines of the file:
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@@
     (company "Filippo Gottardo")
   )
-  (junction (at 114.3 38.1) (diameter 0) (color 0 0 0 0)
+  (junction (at 127 49.53) (diameter 0) (color 0 0 0 0)
   )
   (junction (at 222.25 88.9) (diameter 0) (color 0 0 0 0)
   )
   (junction (at 139.7 92.71) (diameter 0) (color 0 0 0 0)
+  )
+  (junction (at 114.3 26.67) (diameter 0) (color 0 0 0 0)
+  )
+  (junction (at 152.4 38.1) (diameter 0) (color 0 0 0 0)
   )
   (junction (at 120.65 97.79) (diameter 0) (color 0 0 0 0)
@@
     (stroke (width 0) (type default) (color 0 0 0 0))
   )
-  (wire (pts (xy 114.3 38.1) (xy 114.3 40.64))
-    (stroke (width 0) (type default) (color 0 0 0 0))
-  )
   (wire (pts (xy 60.96 68.58) (xy 60.96 66.04))
     (stroke (width 0) (type default) (color 0 0 0 0))
@@
     (stroke (width 0) (type default) (color 0 0 0 0))
   )
-  (wire (pts (xy 118.11 44.45) (xy 120.65 44.45))
-    (stroke (width 0) (type default) (color 0 0 0 0))
-  )
   (wire (pts (xy 59.69 165.1) (xy 59.69 161.29))
     (stroke (width 0) (type default) (color 0 0 0 0))
@@
     (stroke (width 0) (type default) (color 0 0 0 0))
   )
-  (wire (pts (xy 114.3 25.4) (xy 114.3 27.94))
+  (wire (pts (xy 152.4 31.75) (xy 146.685 31.75))
+    (stroke (width 0) (type default) (color 0 0 0 0))
+  )
+  (wire (pts (xy 114.3 25.4) (xy 114.3 26.67))
     (stroke (width 0) (type default) (color 0 0 0 0))
   )
@@
     (stroke (width 0) (type default) (color 0 0 0 0))
   )
+  (wire (pts (xy 114.3 26.67) (xy 114.3 27.94))
+    (stroke (width 0) (type default) (color 0 0 0 0))
+  )
   (wire (pts (xy 120.65 97.79) (xy 152.4 97.79))
     (stroke (width 0) (type default) (color 0 0 0 0))
@@
     (stroke (width 0) (type default) (color 0 0 0 0))
   )
+  (wire (pts (xy 118.11 31.75) (xy 139.065 31.75))
+    (stroke (width 0) (type default) (color 0 0 0 0))
+  )
   (wire (pts (xy 120.65 168.91) (xy 120.65 173.99))
     (stroke (width 0) (type default) (color 0 0 0 0))
@@
     (stroke (width 0) (type default) (color 0 0 0 0))
   )
-  (wire (pts (xy 114.3 35.56) (xy 114.3 38.1))
-    (stroke (width 0) (type default) (color 0 0 0 0))
-  )
-  (wire (pts (xy 118.11 31.75) (xy 139.7 31.75))
+  (wire (pts (xy 127 26.67) (xy 127 40.64))
     (stroke (width 0) (type default) (color 0 0 0 0))
   )
@@
     (stroke (width 0) (type default) (color 0 0 0 0))
   )
+  (wire (pts (xy 114.3 26.67) (xy 127 26.67))
+    (stroke (width 0) (type default) (color 0 0 0 0))
+  )
   (wire (pts (xy 60.96 186.69) (xy 60.96 189.23))
     (stroke (width 0) (type default) (color 0 0 0 0))
@@
     (stroke (width 0) (type default) (color 0 0 0 0))
   )
+  (wire (pts (xy 127 49.53) (xy 127 50.8))
+    (stroke (width 0) (type default) (color 0 0 0 0))
+  )
   (wire (pts (xy 59.69 161.29) (xy 63.5 161.29))
     (stroke (width 0) (type default) (color 0 0 0 0))
@@
     (stroke (width 0) (type default) (color 0 0 0 0))
   )
+  (wire (pts (xy 114.3 49.53) (xy 127 49.53))
+    (stroke (width 0) (type default) (color 0 0 0 0))
+  )
   (wire (pts (xy 38.1 69.85) (xy 38.1 64.77))
     (stroke (width 0) (type default) (color 0 0 0 0))
@@
     (stroke (width 0) (type default) (color 0 0 0 0))
   )
-  (wire (pts (xy 120.65 38.1) (xy 114.3 38.1))
-    (stroke (width 0) (type default) (color 0 0 0 0))
-  )
-  (wire (pts (xy 114.3 48.26) (xy 114.3 50.8))
+  (wire (pts (xy 127 48.26) (xy 127 49.53))
     (stroke (width 0) (type default) (color 0 0 0 0))
   )
@@
     (stroke (width 0) (type default) (color 0 0 0 0))
   )
+  (wire (pts (xy 146.685 44.45) (xy 152.4 44.45))
+    (stroke (width 0) (type default) (color 0 0 0 0))
+  )
   (wire (pts (xy 222.25 88.9) (xy 228.6 88.9))
     (stroke (width 0) (type default) (color 0 0 0 0))
@@
     (stroke (width 0) (type default) (color 0 0 0 0))
   )
+  (wire (pts (xy 130.81 44.45) (xy 139.065 44.45))
+    (stroke (width 0) (type default) (color 0 0 0 0))
+  )
+  (wire (pts (xy 152.4 44.45) (xy 152.4 38.1))
+    (stroke (width 0) (type default) (color 0 0 0 0))
+  )
   (wire (pts (xy 119.38 67.31) (xy 121.92 67.31))
     (stroke (width 0) (type default) (color 0 0 0 0))
@@
     (stroke (width 0) (type default) (color 0 0 0 0))
   )
+  (wire (pts (xy 152.4 38.1) (xy 152.4 31.75))
+    (stroke (width 0) (type default) (color 0 0 0 0))
+  )
   (wire (pts (xy 120.65 97.79) (xy 120.65 110.49))
     (stroke (width 0) (type default) (color 0 0 0 0))
@@
     (stroke (width 0) (type default) (color 0 0 0 0))
   )
-  (wire (pts (xy 120.65 44.45) (xy 120.65 38.1))
+  (wire (pts (xy 114.3 35.56) (xy 114.3 49.53))
     (stroke (width 0) (type default) (color 0 0 0 0))
   )
@@
   )
   (wire (pts (xy 60.96 34.29) (xy 63.5 34.29))
+    (stroke (width 0) (type default) (color 0 0 0 0))
+  )
+  (wire (pts (xy 152.4 38.1) (xy 158.75 38.1))
     (stroke (width 0) (type default) (color 0 0 0 0))
   )
@@
     )
   )
-  (global_label "Manual_mod" (shape bidirectional) (at 139.7 31.75 0) (fields_autoplaced)
+  (global_label "Manual_mod" (shape bidirectional) (at 158.75 38.1 0) (fields_autoplaced)
     (effects (font (size 1.27 1.27)) (justify left))
-    (property "Intersheet References" "${INTERSHEET_REFS}" (id 0) (at 153.785 31.6706 0)
+    (property "Intersheet References" "${INTERSHEET_REFS}" (id 0) (at 172.835 38.0206 0)
       (effects (font (size 1.27 1.27)) (justify left) hide)
     )
@@
     (pin "3")
   )
-  (symbol (lib_id "power:-12V") (at 114.3 50.8 180) (unit 1)
-    (in_bom yes) (on_board yes) (fields_autoplaced)
-    (property "Reference" "#PWR014" (id 0) (at 114.3 53.34 0)
-      (effects (font (size 1.27 1.27)) hide)
-    )
-    (property "Value" "-12V" (id 1) (at 114.3 55.3625 0))
-    (property "Footprint" "" (id 2) (at 114.3 50.8 0)
-      (effects (font (size 1.27 1.27)) hide)
-    )
-    (property "Datasheet" "" (id 3) (at 114.3 50.8 0)
+  (symbol (lib_id "power:-12V") (at 127 50.8 180) (unit 1)
+    (in_bom yes) (on_board yes) (fields_autoplaced)
+    (property "Reference" "#PWR014" (id 0) (at 127 53.34 0)
+      (effects (font (size 1.27 1.27)) hide)
+    )
+    (property "Value" "-12V" (id 1) (at 127 55.3625 0))
+    (property "Footprint" "" (id 2) (at 127 50.8 0)
+      (effects (font (size 1.27 1.27)) hide)
+    )
+    (property "Datasheet" "" (id 3) (at 127 50.8 0)
       (effects (font (size 1.27 1.27)) hide)
     )
@@
     (pin "6")
   )
+  (symbol (lib_id "Device:R") (at 142.875 44.45 90) (unit 1)
+    (in_bom yes) (on_board yes) (fields_autoplaced)
+    (property "Reference" "R11" (id 0) (at 142.875 39.4675 90))
+    (property "Value" "100k" (id 1) (at 142.875 42.2426 90))
+    (property "Footprint" "Resistor_THT:R_Axial_DIN0207_L6.3mm_D2.5mm_P10.16mm_Horizontal" (id 2) (at 142.875 46.228 90)
+      (effects (font (size 1.27 1.27)) hide)
+    )
+    (property "Datasheet" "~" (id 3) (at 142.875 44.45 0)
+      (effects (font (size 1.27 1.27)) hide)
+    )
+    (pin "1")
+    (pin "2")
+  )
   (symbol (lib_id "Device:R_Potentiometer") (at 38.1 156.21 0) (mirror x) (unit 1)
     (in_bom yes) (on_board yes) (fields_autoplaced)
@@
     (pin "3")
   )
+  (symbol (lib_id "Device:R") (at 142.875 31.75 90) (unit 1)
+    (in_bom yes) (on_board yes) (fields_autoplaced)
+    (property "Reference" "R10" (id 0) (at 142.875 26.7675 90))
+    (property "Value" "10k" (id 1) (at 142.875 29.5426 90))
+    (property "Footprint" "Resistor_THT:R_Axial_DIN0207_L6.3mm_D2.5mm_P10.16mm_Horizontal" (id 2) (at 142.875 33.528 90)
+      (effects (font (size 1.27 1.27)) hide)
+    )
+    (property "Datasheet" "~" (id 3) (at 142.875 31.75 0)
+      (effects (font (size 1.27 1.27)) hide)
+    )
+    (pin "1")
+    (pin "2")
+  )
   (symbol (lib_id "Device:R") (at 120.65 177.8 0) (unit 1)
     (in_bom yes) (on_board yes) (fields_autoplaced)
@@
     (pin "2")
   )
-  (symbol (lib_id "Device:R_Potentiometer") (at 114.3 44.45 0) (unit 1)
-    (in_bom yes) (on_board yes) (fields_autoplaced)
-    (property "Reference" "RV7" (id 0) (at 112.522 43.5415 0)
-      (effects (font (size 1.27 1.27)) (justify right))
-    )
-    (property "Value" "1k-Fine" (id 1) (at 112.522 46.3166 0)
-      (effects (font (size 1.27 1.27)) (justify right))
-    )
-    (property "Footprint" "Custom Footprints:RV-90 Potentiometer" (id 2) (at 114.3 44.45 0)
-      (effects (font (size 1.27 1.27)) hide)
-    )
-    (property "Datasheet" "~" (id 3) (at 114.3 44.45 0)
+  (symbol (lib_id "Device:R_Potentiometer") (at 127 44.45 0) (unit 1)
+    (in_bom yes) (on_board yes) (fields_autoplaced)
+    (property "Reference" "RV7" (id 0) (at 125.2221 43.5415 0)
+      (effects (font (size 1.27 1.27)) (justify right))
+    )
+    (property "Value" "10k-Fine" (id 1) (at 125.2221 46.3166 0)
+      (effects (font (size 1.27 1.27)) (justify right))
+    )
+    (property "Footprint" "Custom Footprints:RV-90 Potentiometer" (id 2) (at 127 44.45 0)
+      (effects (font (size 1.27 1.27)) hide)
+    )
+    (property "Datasheet" "~" (id 3) (at 127 44.45 0)
       (effects (font (size 1.27 1.27)) hide)
     )
@@
       (reference "R9") (unit 1) (value "560R") (footprint "Resistor_THT:R_Axial_DIN0207_L6.3mm_D2.5mm_P10.16mm_Horizontal")
     )
+    (path "/9f329818-1dc0-4a6e-8604-709f4943d9ed"
+      (reference "R10") (unit 1) (value "10k") (footprint "Resistor_THT:R_Axial_DIN0207_L6.3mm_D2.5mm_P10.16mm_Horizontal")
+    )
+    (path "/88753d3c-e288-4a8d-a9a1-29448a3cba6a"
+      (reference "R11") (unit 1) (value "100k") (footprint "Resistor_THT:R_Axial_DIN0207_L6.3mm_D2.5mm_P10.16mm_Horizontal")
+    )
     (path "/11373472-8a91-4578-bed7-64a0e1ed98fd"
       (reference "RV1") (unit 1) (value "Volume 1-1k") (footprint "Custom Footprints:RV-90 Potentiometer")
@@
     )
     (path "/f8ff0b15-dcca-43a9-829a-230e008f124a"
-      (reference "RV7") (unit 1) (value "1k-Fine") (footprint "Custom Footprints:RV-90 Potentiometer")
+      (reference "RV7") (unit 1) (value "10k-Fine") (footprint "Custom Footprints:RV-90 Potentiometer")
     )
     (path "/feec861b-a0a8-426a-9539-26f3d3930030"

Commit message: finished ch06 and added appendix
Parts:
- R6, R7: value 220R -> 560R
- R8, R9: value 560R -> 2k2
Changed lines of the file:
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@@
       (effects (font (size 1.27 1.27)) (justify left))
     )
-    (property "Value" "220R" (id 1) (at 141.478 116.1666 0)
+    (property "Value" "560R" (id 1) (at 141.478 116.1666 0)
       (effects (font (size 1.27 1.27)) (justify left))
     )
@@
       (effects (font (size 1.27 1.27)) (justify left))
     )
-    (property "Value" "220R" (id 1) (at 122.428 116.1666 0)
+    (property "Value" "560R" (id 1) (at 122.428 116.1666 0)
       (effects (font (size 1.27 1.27)) (justify left))
     )
@@
       (effects (font (size 1.27 1.27)) (justify left))
     )
-    (property "Value" "560R" (id 1) (at 122.428 179.6666 0)
+    (property "Value" "2k2" (id 1) (at 122.428 179.6666 0)
       (effects (font (size 1.27 1.27)) (justify left))
     )
@@
       (effects (font (size 1.27 1.27)) (justify left))
     )
-    (property "Value" "560R" (id 1) (at 147.828 179.6666 0)
+    (property "Value" "2k2" (id 1) (at 147.828 179.6666 0)
       (effects (font (size 1.27 1.27)) (justify left))
     )
@@
     )
     (path "/1c5ce44e-603d-487b-b527-14e5889da608"
-      (reference "R6") (unit 1) (value "220R") (footprint "Resistor_THT:R_Axial_DIN0207_L6.3mm_D2.5mm_P10.16mm_Horizontal")
+      (reference "R6") (unit 1) (value "560R") (footprint "Resistor_THT:R_Axial_DIN0207_L6.3mm_D2.5mm_P10.16mm_Horizontal")
     )
     (path "/12c66e26-a2e7-4450-ace7-a347ace0f572"
-      (reference "R7") (unit 1) (value "220R") (footprint "Resistor_THT:R_Axial_DIN0207_L6.3mm_D2.5mm_P10.16mm_Horizontal")
+      (reference "R7") (unit 1) (value "560R") (footprint "Resistor_THT:R_Axial_DIN0207_L6.3mm_D2.5mm_P10.16mm_Horizontal")
     )
     (path "/a1bf9496-c225-4809-86d9-f9f15289f8f8"
-      (reference "R8") (unit 1) (value "560R") (footprint "Resistor_THT:R_Axial_DIN0207_L6.3mm_D2.5mm_P10.16mm_Horizontal")
+      (reference "R8") (unit 1) (value "2k2") (footprint "Resistor_THT:R_Axial_DIN0207_L6.3mm_D2.5mm_P10.16mm_Horizontal")
     )
     (path "/ee217293-ddc6-462b-afed-e924309e0558"
-      (reference "R9") (unit 1) (value "560R") (footprint "Resistor_THT:R_Axial_DIN0207_L6.3mm_D2.5mm_P10.16mm_Horizontal")
+      (reference "R9") (unit 1) (value "2k2") (footprint "Resistor_THT:R_Axial_DIN0207_L6.3mm_D2.5mm_P10.16mm_Horizontal")
     )
     (path "/9f329818-1dc0-4a6e-8604-709f4943d9ed"
